File: BrewPi Sensor Boards/RJ-45 v1.1 Top Routed.sch (EAGLE design)
At the start: 6 parts, among them J1 RJ45-8X

Commit message: Update RJ-45 Board Design
Connections:
- net 5V renamed VCC
Other:
- note added: "6 - Door 5 - GND 4 - OneWire Data 3 - VCC (Voltage selected by controller board)"
- note removed: "6 - Door 5 - GND 4 - OneWire 3 - 5v"
Changed lines of the file:
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@@
 <text x="71.12" y="38.1" size="1.778" layer="95">6 - Door
 5 - GND
-4 - OneWire
-3 - 5v</text>
+4 - OneWire Data
+3 - VCC (Voltage selected by controller board)</text>
 </plain>
 <instances>
@@
 </segment>
 </net>
-<net name="5V" class="0">
+<net name="VCC" class="0">
 <segment>
 <wire x1="45.72" y1="53.34" x2="45.72" y2="73.66" width="0.1524" layer="91"/>
