File: ESP8266 BrewPi Boards/D1 - LCD TH Screws.sch (EAGLE design)
At the start: 7 parts, among them J1 RJ45-8X

Commit message: Updating TH Screw board
Parts:
- added C1, C3: 0.1uF, rcl:C-EU050-035X075
- added C2, C4: 1uF, rcl:C-EU050-035X075
- added ONEWIRE_VSEL: (no value), jumper:SJ2WW
Connections:
- new net N$3: J1.3, ONEWIRE_VSEL.2
- net 3V3: now also C3.1, C4.1, ONEWIRE_VSEL.3; no longer J1.3
- net 5V: now also C1.2, C2.2, ONEWIRE_VSEL.1
- net GND: now also C1.1, C2.1, C3.2, C4.2
Other:
- note added: "5 - Door (D7) 4 - GND 3 - OneWire (D6) 2 - 3v3/5v"
- note removed: "5 - Door (D7) 4 - GND 3 - OneWire (D6) 2 - 3v3"
- moved on the sheet: R1
Changed lines of the file:
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@@
 <part name="U$3" library="SparkFun-Boards" library_urn="urn:adsk.eagle:library:509" deviceset="SPARKFUN_LOGIC_LEVEL_CONVERTER" device="" package3d_urn="urn:adsk.eagle:package:37318/1"/>
 <part name="X1" library="con-wago-500" deviceset="W237-4" device=""/>
+<part name="C1" library="rcl" library_urn="urn:adsk.eagle:library:334" deviceset="C-EU" device="050-035X075" package3d_urn="urn:adsk.eagle:package:23677/1" value="0.1uF"/>
+<part name="C2" library="rcl" library_urn="urn:adsk.eagle:library:334" deviceset="C-EU" device="050-035X075" package3d_urn="urn:adsk.eagle:package:23677/1" value="1uF"/>
+<part name="C3" library="rcl" library_urn="urn:adsk.eagle:library:334" deviceset="C-EU" device="050-035X075" package3d_urn="urn:adsk.eagle:package:23677/1" value="0.1uF"/>
+<part name="C4" library="rcl" library_urn="urn:adsk.eagle:library:334" deviceset="C-EU" device="050-035X075" package3d_urn="urn:adsk.eagle:package:23677/1" value="1uF"/>
+<part name="ONEWIRE_VSEL" library="jumper" library_urn="urn:adsk.eagle:library:252" deviceset="SJ2W" device="W" package3d_urn="urn:adsk.eagle:package:15476/1"/>
 </parts>
 <sheets>
@@
 4 - GND
 3 - OneWire (D6)
-2 - 3v3</text>
+2 - 3v3/5v</text>
 <text x="50.8" y="30.48" size="1.778" layer="97">1 - +5v
 2 - GND</text>
@@
 <attribute name="VALUE" x="17.78" y="53.848" size="1.778" layer="96" rot="R180"/>
 </instance>
-<instance part="R1" gate="G$1" x="33.02" y="35.56" smashed="yes" rot="R90">
-<attribute name="NAME" x="31.5214" y="31.75" size="1.778" layer="95" rot="R90"/>
-<attribute name="VALUE" x="36.322" y="31.75" size="1.778" layer="96" rot="R90"/>
+<instance part="R1" gate="G$1" x="38.1" y="40.64" smashed="yes" rot="R180">
+<attribute name="NAME" x="41.91" y="39.1414" size="1.778" layer="95" rot="R180"/>
+<attribute name="VALUE" x="41.91" y="43.942" size="1.778" layer="96" rot="R180"/>
 </instance>
 <instance part="RELAY" gate="-1" x="20.32" y="76.2" smashed="yes">
@@
 <attribute name="VALUE" x="111.76" y="41.783" size="1.778" layer="96" rot="R180"/>
 <attribute name="NAME" x="109.22" y="37.211" size="1.778" layer="95"/>
+</instance>
+<instance part="C1" gate="G$1" x="83.82" y="53.34" smashed="yes">
+<attribute name="NAME" x="85.344" y="53.721" size="1.778" layer="95"/>
+<attribute name="VALUE" x="85.344" y="48.641" size="1.778" layer="96"/>
+</instance>
+<instance part="C2" gate="G$1" x="91.44" y="53.34" smashed="yes">
+<attribute name="NAME" x="92.964" y="53.721" size="1.778" layer="95"/>
+<attribute name="VALUE" x="92.964" y="48.641" size="1.778" layer="96"/>
+</instance>
+<instance part="C3" gate="G$1" x="73.66" y="38.1" smashed="yes">
+<attribute name="NAME" x="75.184" y="38.481" size="1.778" layer="95"/>
+<attribute name="VALUE" x="75.184" y="33.401" size="1.778" layer="96"/>
+</instance>
+<instance part="C4" gate="G$1" x="81.28" y="38.1" smashed="yes">
+<attribute name="NAME" x="82.804" y="38.481" size="1.778" layer="95"/>
+<attribute name="VALUE" x="82.804" y="33.401" size="1.778" layer="96"/>
+</instance>
+<instance part="ONEWIRE_VSEL" gate="G$1" x="33.02" y="25.4" smashed="yes">
+<attribute name="NAME" x="35.56" y="25.781" size="1.778" layer="95"/>
+<attribute name="VALUE" x="35.56" y="23.495" size="1.778" layer="96"/>
 </instance>
 </instances>
@@
 <segment>
 <pinref part="U$1" gate="G$1" pin="GND"/>
-<wire x1="68.58" y1="55.88" x2="73.66" y2="55.88" width="0.1524" layer="91"/>
-<wire x1="73.66" y1="55.88" x2="73.66" y2="50.8" width="0.1524" layer="91"/>
-<wire x1="73.66" y1="50.8" x2="73.66" y2="43.18" width="0.1524" layer="91"/>
-<wire x1="73.66" y1="43.18" x2="68.58" y2="43.18" width="0.1524" layer="91"/>
 <pinref part="X" gate="-2" pin="KL"/>
 <wire x1="68.58" y1="38.1" x2="68.58" y2="43.18" width="0.1524" layer="91"/>
@@
 <pinref part="U$3" gate="G$1" pin="GND"/>
 <wire x1="99.06" y1="66.04" x2="78.74" y2="66.04" width="0.1524" layer="91"/>
-<wire x1="78.74" y1="66.04" x2="78.74" y2="50.8" width="0.1524" layer="91"/>
-<wire x1="78.74" y1="50.8" x2="78.74" y2="45.72" width="0.1524" layer="91"/>
-<wire x1="78.74" y1="45.72" x2="93.98" y2="45.72" width="0.1524" layer="91"/>
+<wire x1="78.74" y1="66.04" x2="78.74" y2="55.88" width="0.1524" layer="91"/>
+<wire x1="78.74" y1="55.88" x2="78.74" y2="45.72" width="0.1524" layer="91"/>
+<wire x1="78.74" y1="45.72" x2="86.36" y2="45.72" width="0.1524" layer="91"/>
+<wire x1="86.36" y1="45.72" x2="93.98" y2="45.72" width="0.1524" layer="91"/>
 <wire x1="93.98" y1="45.72" x2="134.62" y2="45.72" width="0.1524" layer="91"/>
-<wire x1="73.66" y1="50.8" x2="78.74" y2="50.8" width="0.1524" layer="91"/>
-<junction x="73.66" y="50.8"/>
-<junction x="78.74" y="50.8"/>
 <pinref part="X1" gate="-1" pin="KL"/>
 <wire x1="104.14" y1="22.86" x2="93.98" y2="22.86" width="0.1524" layer="91"/>
@@
 <wire x1="132.08" y1="66.04" x2="134.62" y2="66.04" width="0.1524" layer="91"/>
 <wire x1="134.62" y1="66.04" x2="134.62" y2="45.72" width="0.1524" layer="91"/>
+<wire x1="68.58" y1="55.88" x2="78.74" y2="55.88" width="0.1524" layer="91"/>
+<junction x="78.74" y="55.88"/>
+<wire x1="68.58" y1="43.18" x2="78.74" y2="43.18" width="0.1524" layer="91"/>
+<wire x1="78.74" y1="43.18" x2="78.74" y2="45.72" width="0.1524" layer="91"/>
+<junction x="78.74" y="45.72"/>
+<pinref part="C1" gate="G$1" pin="1"/>
+<wire x1="83.82" y1="55.88" x2="78.74" y2="55.88" width="0.1524" layer="91"/>
+<pinref part="C2" gate="G$1" pin="1"/>
+<wire x1="91.44" y1="55.88" x2="83.82" y2="55.88" width="0.1524" layer="91"/>
+<junction x="83.82" y="55.88"/>
+<pinref part="C3" gate="G$1" pin="2"/>
+<pinref part="C4" gate="G$1" pin="2"/>
+<wire x1="73.66" y1="33.02" x2="81.28" y2="33.02" width="0.1524" layer="91"/>
+<wire x1="81.28" y1="33.02" x2="86.36" y2="33.02" width="0.1524" layer="91"/>
+<junction x="81.28" y="33.02"/>
+<wire x1="86.36" y1="33.02" x2="86.36" y2="45.72" width="0.1524" layer="91"/>
+<junction x="86.36" y="45.72"/>
 </segment>
 </net>
@@
 <wire x1="30.48" y1="60.96" x2="30.48" y2="58.42" width="0.1524" layer="91"/>
 <wire x1="30.48" y1="58.42" x2="35.56" y2="58.42" width="0.1524" layer="91"/>
-<wire x1="71.12" y1="48.26" x2="96.52" y2="48.26" width="0.1524" layer="91"/>
+<wire x1="71.12" y1="48.26" x2="83.82" y2="48.26" width="0.1524" layer="91"/>
+<wire x1="83.82" y1="48.26" x2="91.44" y2="48.26" width="0.1524" layer="91"/>
+<wire x1="91.44" y1="48.26" x2="96.52" y2="48.26" width="0.1524" layer="91"/>
 <wire x1="96.52" y1="48.26" x2="137.16" y2="48.26" width="0.1524" layer="91"/>
 <wire x1="137.16" y1="48.26" x2="137.16" y2="68.58" width="0.1524" layer="91"/>
@@
 <label x="99.06" y="27.94" size="1.778" layer="95"/>
 <label x="27.94" y="60.96" size="1.778" layer="95"/>
+<wire x1="30.48" y1="33.02" x2="30.48" y2="58.42" width="0.1524" layer="91"/>
+<junction x="30.48" y="58.42"/>
+<pinref part="C1" gate="G$1" pin="2"/>
+<junction x="83.82" y="48.26"/>
+<pinref part="C2" gate="G$1" pin="2"/>
+<junction x="91.44" y="48.26"/>
+<wire x1="30.48" y1="33.02" x2="33.02" y2="33.02" width="0.1524" layer="91"/>
+<pinref part="ONEWIRE_VSEL" gate="G$1" pin="1"/>
+<wire x1="33.02" y1="33.02" x2="33.02" y2="30.48" width="0.1524" layer="91"/>
+<label x="33.02" y="33.02" size="1.778" layer="95"/>
 </segment>
 </net>
 <net name="3V3" class="2">
 <segment>
-<pinref part="U$1" gate="G$1" pin="3V3"/>
-<wire x1="43.18" y1="53.34" x2="40.64" y2="53.34" width="0.1524" layer="91"/>
-<wire x1="40.64" y1="53.34" x2="40.64" y2="30.48" width="0.1524" layer="91"/>
-<pinref part="R1" gate="G$1" pin="1"/>
-<wire x1="27.94" y1="38.1" x2="27.94" y2="30.48" width="0.1524" layer="91"/>
-<wire x1="27.94" y1="30.48" x2="33.02" y2="30.48" width="0.1524" layer="91"/>
-<wire x1="40.64" y1="30.48" x2="33.02" y2="30.48" width="0.1524" layer="91"/>
-<junction x="33.02" y="30.48"/>
 <pinref part="U$3" gate="G$1" pin="LV"/>
 <wire x1="99.06" y1="68.58" x2="81.28" y2="68.58" width="0.1524" layer="91"/>
-<wire x1="81.28" y1="68.58" x2="81.28" y2="25.4" width="0.1524" layer="91"/>
-<wire x1="81.28" y1="25.4" x2="40.64" y2="25.4" width="0.1524" layer="91"/>
-<wire x1="40.64" y1="25.4" x2="40.64" y2="30.48" width="0.1524" layer="91"/>
-<junction x="40.64" y="30.48"/>
-<pinref part="J1" gate="G$1" pin="3"/>
-<wire x1="20.32" y1="38.1" x2="27.94" y2="38.1" width="0.1524" layer="91"/>
-<label x="20.32" y="38.1" size="1.778" layer="95"/>
+<wire x1="81.28" y1="68.58" x2="81.28" y2="40.64" width="0.1524" layer="91"/>
+<pinref part="U$1" gate="G$1" pin="3V3"/>
+<pinref part="R1" gate="G$1" pin="1"/>
+<wire x1="43.18" y1="40.64" x2="43.18" y2="53.34" width="0.1524" layer="91"/>
+<wire x1="43.18" y1="40.64" x2="73.66" y2="40.64" width="0.1524" layer="91"/>
+<junction x="43.18" y="40.64"/>
+<pinref part="C3" gate="G$1" pin="1"/>
+<wire x1="73.66" y1="40.64" x2="81.28" y2="40.64" width="0.1524" layer="91"/>
+<junction x="73.66" y="40.64"/>
+<pinref part="C4" gate="G$1" pin="1"/>
+<junction x="81.28" y="40.64"/>
+<pinref part="ONEWIRE_VSEL" gate="G$1" pin="3"/>
+<wire x1="43.18" y1="40.64" x2="43.18" y2="20.32" width="0.1524" layer="91"/>
+<wire x1="43.18" y1="20.32" x2="33.02" y2="20.32" width="0.1524" layer="91"/>
+<label x="35.56" y="20.32" size="1.778" layer="95"/>
 </segment>
 </net>
@@
 </segment>
 </net>
+<net name="N$3" class="0">
+<segment>
+<pinref part="J1" gate="G$1" pin="3"/>
+<wire x1="20.32" y1="38.1" x2="25.4" y2="38.1" width="0.1524" layer="91"/>
+<pinref part="ONEWIRE_VSEL" gate="G$1" pin="2"/>
+<wire x1="25.4" y1="38.1" x2="25.4" y2="25.4" width="0.1524" layer="91"/>
+<wire x1="25.4" y1="25.4" x2="27.94" y2="25.4" width="0.1524" layer="91"/>
+<label x="20.32" y="38.1" size="1.778" layer="95"/>
+</segment>
+</net>
 </nets>
 </sheet>
 </sheets>
+<errors>
+</errors>
 </schematic>
 </drawing>

Commit message: Updating board designs and adding DirtyPCB Links
Parts:
- J1: device con-tycoelectronics:RJ45-8X -> Donnie:RJ45-8X
Changed lines of the file:
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@@
 <layer number="59" name="tCarbon" color="7" fill="1" visible="no" active="no"/>
 <layer number="60" name="bCarbon" color="7" fill="1" visible="no" active="no"/>
+<layer number="88" name="SimResults" color="9" fill="1" visible="yes" active="yes"/>
+<layer number="89" name="SimProbes" color="9" fill="1" visible="yes" active="yes"/>
 <layer number="90" name="Modules" color="5" fill="1" visible="yes" active="yes"/>
 <layer number="91" name="Nets" color="2" fill="1" visible="yes" active="yes"/>
@@
 <layer number="230" name="230bmp" color="7" fill="1" visible="yes" active="yes"/>
 <layer number="231" name="231bmp" color="7" fill="1" visible="yes" active="yes"/>
+<layer number="232" name="Eagle3D_PG2" color="7" fill="1" visible="no" active="no"/>
+<layer number="233" name="Eagle3D_PG3" color="7" fill="1" visible="no" active="no"/>
 <layer number="248" name="Housing" color="7" fill="1" visible="yes" active="yes"/>
 <layer number="249" name="Edge" color="7" fill="1" visible="yes" active="yes"/>
@@
 <part name="U$1" library="1455413453956-wemos" deviceset="WEMOS" device=""/>
 <part name="X" library="con-wago-500" deviceset="W237-102" device="" value="PWR"/>
-<part name="J1" library="con-tycoelectronics" library_urn="urn:adsk.eagle:library:193" deviceset="RJ45" device="" package3d_urn="urn:adsk.eagle:package:10660/1" technology="-8X"/>
+<part name="J1" library="Donnie" deviceset="RJ45" device="" package3d_urn="urn:adsk.eagle:package:10660/1" technology="-8X"/>
 <part name="R1" library="rcl" library_urn="urn:adsk.eagle:library:334" deviceset="R-US_" device="0309/12" package3d_urn="urn:adsk.eagle:package:23571/1" value="4.7k"/>
 <part name="RELAY" library="con-wago-500" deviceset="W237-4" device=""/>
