File: ESP8266 BrewPi Boards/D1 - SMD.sch (EAGLE design)
At the start: 18 parts, among them J1 RJ45-8X, Q1 BSS123, Q2 BSS123

Commit message: Add solder bridge to SMD board design
Parts:
- added OW_VSEL: (no value), jumper:SJ2W
Connections:
- net 3V3: now also OW_VSEL.3
- net 5V: now also OW_VSEL.1
- net OW_VCC: now also OW_VSEL.2
Changed lines of the file:
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@@
 <part name="P+1" library="supply1" library_urn="urn:adsk.eagle:library:371" deviceset="+5V" device=""/>
 <part name="ONEWIRE_VSEL" library="Donnie" deviceset="JP2E" device="NOLABEL"/>
+<part name="OW_VSEL" library="jumper" library_urn="urn:adsk.eagle:library:252" deviceset="SJ2W" device="" package3d_urn="urn:adsk.eagle:package:15474/1"/>
 </parts>
 <sheets>
@@
 <attribute name="NAME" x="22.86" y="13.97" size="1.778" layer="95" rot="R180"/>
 <attribute name="VALUE" x="22.86" y="23.495" size="1.778" layer="96" rot="R180"/>
+</instance>
+<instance part="OW_VSEL" gate="G$1" x="22.86" y="5.08" smashed="yes" rot="R180">
+<attribute name="NAME" x="20.32" y="4.699" size="1.778" layer="95" rot="R180"/>
+<attribute name="VALUE" x="20.32" y="6.985" size="1.778" layer="96" rot="R180"/>
 </instance>
 </instances>
@@
 <wire x1="35.56" y1="15.24" x2="25.4" y2="15.24" width="0.1524" layer="91"/>
 <label x="27.94" y="15.24" size="1.778" layer="95"/>
+<wire x1="35.56" y1="15.24" x2="35.56" y2="0" width="0.1524" layer="91"/>
+<junction x="35.56" y="15.24"/>
+<pinref part="OW_VSEL" gate="G$1" pin="1"/>
+<wire x1="35.56" y1="0" x2="22.86" y2="0" width="0.1524" layer="91"/>
 </segment>
 <segment>
@@
 <junction x="43.18" y="25.4"/>
 <label x="25.4" y="20.32" size="1.778" layer="95"/>
+<wire x1="43.18" y1="20.32" x2="43.18" y2="10.16" width="0.1524" layer="91"/>
+<junction x="43.18" y="20.32"/>
+<pinref part="OW_VSEL" gate="G$1" pin="3"/>
+<wire x1="43.18" y1="10.16" x2="22.86" y2="10.16" width="0.1524" layer="91"/>
 </segment>
 </net>
@@
 <wire x1="30.48" y1="38.1" x2="22.86" y2="38.1" width="0.1524" layer="91"/>
 <label x="27.94" y="17.78" size="1.778" layer="95"/>
-</segment>
-</net>
+<pinref part="OW_VSEL" gate="G$1" pin="2"/>
+<wire x1="30.48" y1="17.78" x2="30.48" y2="5.08" width="0.1524" layer="91"/>
+<wire x1="30.48" y1="5.08" x2="27.94" y2="5.08" width="0.1524" layer="91"/>
+<junction x="30.48" y="17.78"/>
+</segment>
+</net>
